File: Maze_kiCad/Maze_kiCad.kicad_pcb (KiCad board)
At the start: 2 copper layers, 150 x 100 mm, 39 parts, among them J1 Screw_Terminal, J10 pins: 42_41_40_39_38_37, J11 gnd_gnd_45_0_35_36, J12 Vcc/Gnd, J2 motor2, J3 motor1, J4 Vmm/Mode, J5 INT/ADO/XCL/XDA, J6 GND, J7 IR Receiver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

Commit message: Final maze robot pcb and gerber files
Routing:
- net /ir_sensor_6: track 56.9 -> 70.0 mm
- net Net-(D1-RA): track 141.6 -> 139.8 mm
- net VCC: track 315.6 -> 317.4 mm
- net /ir_sensor_4: track 50.4 -> 48.7 mm
- net Net-(J9-Pin_4): track 43.6 -> 44.9 mm
- net Net-(J9-Pin_5): track 39.5 -> 38.4 mm
- net Net-(D1-GA): track 111.5 -> 110.8 mm
- added copper zone on F.Cu, net GND
Other:
- board text added: "Bill Tsolakidis"
